File: MasonJarTop.kicad_pcb (KiCad board)
At the start: 2 copper layers, 65.6 x 65.6 mm, 17 parts, among them P1 CONN_01X02, P2 Loop Mounting Hole, P3 Loop Mounting Hole

Commit message: Finished layout.
Other:
- board text added: "DPW 2016"
Changed lines of the file:
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@@
     (area 90.124847 75.824847 155.875153 141.575153)
     (thickness 1.6)
-    (drawings 1)
+    (drawings 2)
     (tracks 34)
     (zones 0)
@@
     (nets 10)
   )
-  (page A4)
+  (page USLetter)
   (layers
     (0 F.Cu signal)
@@
     (pad_to_mask_clearance 0.2)
     (aux_axis_origin 0 0)
-    (visible_elements FFFFFF7F)
+    (visible_elements 7FFFFFFF)
     (pcbplotparams
-      (layerselection 0x00030_80000001)
+      (layerselection 0x010f0_80000001)
       (usegerberextensions false)
       (excludeedgelayer true)
@@
       (outputformat 1)
       (mirror false)
-      (drillshape 1)
+      (drillshape 0)
       (scaleselection 1)
-      (outputdirectory ""))
+      (outputdirectory Gerbers/))
   )
   (net 0 "")
@@
     )
   )
+  (gr_text "DPW 2016" (at 123.1 96.2) (layer F.SilkS)
+    (effects (font (size 1.5 1.5) (thickness 0.3)))
+  )
   (gr_circle (center 123 108.7) (end 155.8 108.8) (layer Edge.Cuts) (width 0.15))
